File: slimevr-hw/slimevr-hw.kicad_pcb (KiCad board)
At the start: 2 copper layers, 30 x 32 mm, 44 parts, among them J1 USB_C_Receptacle_USB2.0_16P, J2 电池接口, Q1 SI2301, SW1 TS-1088-AR02016, SW2 TS-1088-AR02016, U1 ESP32-C3-WROOM-02-N4, U2 ME6212C33M5G, U3 TP4054, U4 HX MSK12C02-HB, U5 QMC6309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

Commit message: update: layout完成
Parts:
- Q1: value SI2301 -> SOT-23-3_L2.9-W1.6-P1.90-LS2.8-BR
- SW1, SW2: value TS-1088-AR02016 -> SW-SMD_L3.9-W3.0-P4.45
- U2: value ME6212C33M5G -> SOT-23-5_L3.0-W1.7-P0.95-LS2.8-BL
- U3: value TP4054 -> TSOT-23-5_L2.9-W1.6-P0.95-LS2.8-BR
- U4: value HX MSK12C02-HB -> SW-SMD_MSK12C02-HB
- U6: value LSM6DSRTR -> LGA-14_L3.0-W2.5-P0.50-BR
- moved R2 99.1 mm to (125.2, 81.3), turned to 90 degrees
- moved J2 96.8 mm to (122.6, 83.2), turned to 180 degrees
- moved D1 96.3 mm to (125.7, 79.0)
- moved Q1 91.4 mm to (121.7, 79.5)
- moved D3 73.9 mm to (113.5, 70.0), turned to 180 degrees
- moved U4 72.7 mm to (114.8, 83.5)
- moved R14 72.6 mm to (113.5, 71.0), turned to 180 degrees
- moved D4 71.6 mm to (113.5, 68.8), turned to 180 degrees
- moved C3 70.5 mm to (121.0, 76.0)
- moved R15 68.8 mm to (113.5, 67.8), turned to 180 degrees
- moved C6 68.7 mm to (115.0, 76.5), turned to -90 degrees
- moved R10 68.5 mm to (115.0, 78.8), turned to 180 degrees
- moved U2 65.6 mm to (117.7, 76.9)
- moved C10 64.6 mm to (125.5, 84.0), turned to 90 degrees
- moved U3 64.4 mm to (128.5, 83.8), turned to 180 degrees
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Routing:
- net +3.3V: track 0.00 -> 75.2 mm, vias 0 -> 4
- net /SCL: track 0.00 -> 51.2 mm, vias 0 -> 3
- net /SDA: track 0.00 -> 44.6 mm
- net +BATT: track 0.00 -> 43.1 mm, vias 0 -> 1
- net +5V: track 0.00 -> 27.9 mm, vias 0 -> 2
- net /INT2: track 0.00 -> 17.8 mm, vias 0 -> 4
- net /INT1: track 0.00 -> 14.7 mm, vias 0 -> 2
- net /EN: track 0.00 -> 13.2 mm, vias 0 -> 2
- net Net-(D1-K): track 0.00 -> 12.0 mm
- net /BOOT: track 0.00 -> 8.67 mm, vias 0 -> 2
- net /LED1: track 0.00 -> 7.64 mm
- net Net-(U1-IO4): track 0.00 -> 5.60 mm
- net Net-(U2-CE): track 0.00 -> 5.01 mm
- net Net-(U6-CS): track 0.00 -> 4.04 mm
- net Net-(R10-Pad2): track 0.00 -> 3.84 mm
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- added copper zone on B.Cu, net GND
- added copper zone on F.Cu, net GND
Other:
- outline, holes or cut-outs redrawn
- board text added: "- +"
- board text added: "BOOT"
- board text added: "RST"

Commit message: update: 同步更改
Parts:
- D2, D3, D4: footprint LED_SMD:LED_0402_1005Metric -> LED_SMD:LED_0603_1608Metric
- Q1: value SOT-23-3_L2.9-W1.6-P1.90-LS2.8-BR -> SI2301
- R3, R4: value 470K -> 1M
- SW1, SW2: value SW-SMD_L3.9-W3.0-P4.45 -> TS-1088-AR02016
- U2: value SOT-23-5_L3.0-W1.7-P0.95-LS2.8-BL -> ME6212C33M5G
- U3: value TSOT-23-5_L2.9-W1.6-P0.95-LS2.8-BR -> TP4054
- U4: value SW-SMD_MSK12C02-HB -> HX MSK12C02-HB
- U6: value LGA-14_L3.0-W2.5-P0.50-BR -> LSM6DSRTR
- moved D1 1.10 mm to (125.2, 78.0)
- moved R14 0.75 mm to (113.5, 71.8)
- moved D2 0.56 mm to (126.8, 80.5)
- moved D3 0.51 mm to (113.5, 70.5)
- moved R6 0.51 mm to (110.8, 68.2)
- moved D4 0.25 mm to (113.5, 69.0)
Routing:
- net +5V: track 27.9 -> 29.4 mm
