File: slimevr-hw/slimevr-hw.kicad_sch (KiCad schematic)
At the start: 52 parts, among them J1 USB_C_Receptacle_USB2.0_16P, J2 电池接口, Q1 SI2301, SW2 TS-1088-AR02016, SW3 TS-1088-AR02016, U1 ESP32-C3-WROOM-02-N4, U2 BQ24040DSQR, U3 LSM6DSRTR, U4 ME6212C33M5G, U5 SK12D07VG5, U6 QMC6309

Commit message: update: 改改不合理的地方
Parts:
- removed U5: SK12D07VG5, kicad_api_lib:SK12D07VG5, symbol SK12D07VG5:SK12D07VG5_C3020419
- added U7: HX MSK12C02-HB, kicad_api_lib:HX MSK12C02-HB, symbol HX MSK12C02-HB:HX MSK12C02-HB
- R15, R16: value 10K -> 4.7K
- R3, R4: value 100K -> 1M
Connections:
- net GND: now also U7.3, U7.4
- net at R9.2: now also U7.1
- net at U4.3 (CE): now also U7.2
Other:
- moved on the sheet: R9

Commit message: add: 软件固件
Parts:
- removed D6, D7: LED, symbol Device:LED
- removed R20, R21: 1K, symbol Device:R
- C1, C10, C12, C5, C8, C9: footprint (none) -> Capacitor_SMD:C_0402_1005Metric
- C11, C13, C2, C3, C4, C6, C7: footprint (none) -> Capacitor_SMD:C_0603_1608Metric
- D1, D2, D4, D5: footprint (none) -> LED_SMD:LED_0402_1005Metric
- R1, R10, R11, R12, R13, R14, R15, R16, R17, R18, R19, R2, R5, R6, R7, R8, R9: footprint (none) -> Resistor_SMD:R_0402_1005Metric
- R3, R4: value 1M -> 470K; footprint (none) -> Resistor_SMD:R_0402_1005Metric
Connections:
- net LED2: no longer names the net of U1.10 (IO10)
- net LED3: no longer names the net of U1.15 (IO3)
- no-connect marks 9 -> 11
Other:
- moved on the sheet: D4, D5, R18, R19

Commit message: update: 充电方案换更简单的
Parts:
- removed C2, C3: 1uF, Capacitor_SMD:C_0603_1608Metric, symbol Device:C
- removed D1: LED, LED_SMD:LED_0402_1005Metric, symbol Device:LED
- removed D3: SS14, Diode_SMD:D_SMA, symbol Diode:SS14
- removed R10: 10K, Resistor_SMD:R_0402_1005Metric, symbol Device:R
- removed R5, R6: 1.5K, Resistor_SMD:R_0402_1005Metric, symbol Device:R
- removed R7: 2K, Resistor_SMD:R_0402_1005Metric, symbol Device:R
- removed R8: 1K, Resistor_SMD:R_0402_1005Metric, symbol Device:R
- removed U2: BQ24040DSQR, kicad_api_lib:BQ24040DSQR, symbol BQ24040DSQR:TI-BQ24040DSQ10-1500X900TP
- added C10: 10uF, Capacitor_SMD:C_0603_1608Metric, symbol Device:C
- added C12: 4.7uF, Capacitor_SMD:C_0603_1608Metric, symbol Device:C
- added D1: 1N5819WS, Diode_SMD:D_SOD-323, symbol Diode:1N5819WS
- added R13: 2K, Resistor_SMD:R_0402_1005Metric, symbol Device:R
- added R9: 1K, Resistor_SMD:R_0402_1005Metric, symbol Device:R
- added U3: TP4054, kicad_api_lib:TP4054, symbol TP4054:TP4054_C668215
- U1: footprint kicad_api_lib:ESP32-C3-WROOM-02-N4 -> kicad_api_lib:ESP-WROOM-02-N4
- renumbered C5 to C1, C9 to C11, C10 to C13, C1 to C2, C13 to C3, C6 to C4, C7 to C5, C4 to C6, C8 to C7, C12 to C8, C11 to C9, D4 to D3, D5 to D4, R12 to R1, R9 to R10, R17 to R11, R15 to R12, R18 to R14, R19 to R15, R14 to R2, R11 to R5, R13 to R6, R1 to R7, R2 to R8, SW2 to SW1, SW3 to SW2, U4 to U2, U7 to U4, U6 to U5, U3 to U6
Connections:
- net +5V: now also C12.1, D1.2 (A), R9.2, U3.4 (VCC)
- net +BATT: now also C10.1, U3.3 (BAT)
- net GND: now also C10.2, C12.2, R13.1, U3.2 (GND)
- net at D2.2 (A): now also R9.1
- net at D2.1 (K): now also U3.1 (CHRG)
- net at C3.1, Q1.2 (S), R10.1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: now also D1.1 (K)
- new net: R13.2, U3.5 (PROG)
- no-connect marks 11 -> 10

Commit message: update: 同步更改
Parts:
- D2, D3, D4: footprint LED_SMD:LED_0402_1005Metric -> LED_SMD:LED_0603_1608Metric
- R3, R4: value 470K -> 1M
